File: Documentation/OpenPLCVersion2.0/KiCAD_Files/Main_Board/OpenPLC_Kicad_Single_Strip_Unordered.kicad_pcb (KiCad board)
At the start: 2 copper layers, 114.8 x 85.2 mm, 161 parts, among them CON1 BARREL_JACK, CON2 AVR-ISP-10, IC1 ATMEGA16-P, P1 LM2596, P10 PortC_B, P11 PortD_B, P12 PortA_M, P13 PortB_M, P14 PortC_M, P15 PortD_M, P16 PortA_FM, P2 CONN_02X04, P3 PortA, P4 PortB, P5 PortC, P6 PortD, P7 Max232, P8 PortB_B, P9 PortA_B, SW1 SW_PUSH, U1 7805, Y1 16Mhz

Commit message: Updated Libraries
Parts:
- removed the REF*** at (104.8, 69.1)
- removed the REF*** at (104.9, 78.5)
- added D36: RX, LEDs:LED_0805, F.Cu at (197.1, 54.9)
- added D37: TX, LEDs:LED_0805, F.Cu at (201.4, 54.9)
- added R35: 1K, Resistors_SMD:R_0805, B.Cu at (192.8, 55.9)
- added R36: 1K, Resistors_SMD:R_0805, B.Cu at (199.5, 58.5)
- added REF***: OSHW-Logo2_9.8x8mm_SilkScreen, Symbols:OSHW-Logo2_9.8x8mm_SilkScreen, F.Cu at (99.7, 74.5)
Routing:
- net /TX: track 52.2 -> 68.5 mm
- net /RX: track 57.0 -> 68.4 mm
- net GND: track 423.9 -> 415.1 mm
- net 5V: track 283.7 -> 291.3 mm
- net 12V: track 217.6 -> 212.8 mm, vias 1 -> 0
- net Net-(D37-Pad2): track 0.00 -> 3.78 mm, vias 0 -> 1
- net Net-(D36-Pad2): track 0.00 -> 2.78 mm, vias 0 -> 1
Other:
- net class PWR_2 added: clearance 0.25, trace_width 1, via_dia 1, via_drill 0.6
