File: Resources/OpenPLCVersion2/KiCAD_Files/Main_Board/OpenPLC_V2.kicad_pcb (KiCad board)
At the start: 2 copper layers, 114.8 x 85.2 mm, 42 parts, among them CON1 BARREL_JACK, CON2 AVR-ISP-10, IC1 ATMEGA16-P, J1 Conn_01x04, J2 Conn_01x04, J3 Conn_01x04, J4 Conn_01x04, P10 PortC_B, P11 PortD_B, P12 PortA_M, P13 PortB_M, P14 PortC_M, P15 PortD_M, P3 PortA, P4 PortB, P5 PortC, P6 PortD, P7 Max232, P8 PortB_B, P9 PortA_B, SW1 SW_PUSH, U1 7805, Y1 16Mhz

Commit message: versioning and finalised V 1.3
Parts:
- removed 1N5822: D_Schottky, Diodes_THT:D_DO-201_P12.70mm_Horizontal
- removed CON1: BARREL_JACK, Connectors:BARREL_JACK
- removed P3: PortA, Terminal_Blocks:TerminalBlock_Pheonix_MKDS1.5-12pol
- removed R1, R2: R, Resistors_THT:R_Axial_DIN0207_L6.3mm_D2.5mm_P10.16mm_Horizontal
- removed Reg1: LM2596, TO_SOT_Packages_THT:TO-220-5_Vertical
- added D3: MBR340, Diodes_THT:D_DO-201AD_P15.24mm_Horizontal, F.Cu at (120.4, 107.7)
- added D4: D_Schottky, Diodes_THT:D_DO-201AD_P12.70mm_Horizontal, F.Cu at (106.7, 119.4)
- added J5: Screw_Terminal_01x04, TerminalBlocks_Phoenix:TerminalBlock_Phoenix_MKDS1.5-4pol, F.Cu at (111.0, 44.7)
- added J6: Screw_Terminal_01x08, TerminalBlocks_Phoenix:TerminalBlock_Phoenix_MKDS1.5-8pol, F.Cu at (156.0, 44.7)
- added REF***: OSHW-Logo2_9.8x8mm_SilkScreen, Symbols:OSHW-Logo2_9.8x8mm_SilkScreen, F.Cu at (128.5, 73.7)
- added Regulator1: 24 to 12, TO_SOT_Packages_THT:TO-220-5_Horizontal, F.Cu at (115.3, 109.2)
- added powerIn1: 24V, TerminalBlocks_Phoenix:TerminalBlock_Phoenix_MKDS1.5-2pol, F.Cu at (96.0, 118.9)
- CON2: footprint Connect:IDC_Header_Straight_10pins -> IDC:IDC-Header_2x05_Pitch2.54mm_Straight
- Cin1: value CP -> 100uf
- Cout1: value CP -> 1000uf; footprint Capacitors_THT:CP_Radial_D8.0mm_P3.50mm -> Capacitors_THT:CP_Radial_D10.0mm_P5.00mm
- D1: footprint Diodes_ThroughHole:Diode_DO-41_SOD81_Horizontal_RM10 -> Diodes_THT:D_DO-41_SOD81_P10.16mm_Horizontal
- L1: footprint Choke_Axial_ThroughHole:Choke_Horizontal_RM10mm -> Inductors_SMD:L_Fastron_PISR_Handsoldering
- P10, P11, P8: footprint Socket_Strips:Socket_Strip_Straight_1x08 -> Socket_Strips:Socket_Strip_Straight_1x08_Pitch2.54mm
- P12: footprint Pin_Headers:Pin_Header_Straight_1x12 -> Pin_Headers:Pin_Header_Straight_1x12_Pitch2.54mm
- P13, P14, P15: footprint Pin_Headers:Pin_Header_Straight_1x08 -> Pin_Headers:Pin_Header_Straight_1x08_Pitch2.54mm
- P4, P5, P6: footprint Terminal_Blocks:TerminalBlock_Pheonix_MKDS1.5-8pol -> TerminalBlocks_Phoenix:TerminalBlock_Phoenix_MKDS1.5-8pol
- P7: footprint Socket_Strips:Socket_Strip_Angled_1x04 -> Socket_Strips:Socket_Strip_Angled_1x04_Pitch2.54mm
- P9: footprint Socket_Strips:Socket_Strip_Straight_1x12 -> Socket_Strips:Socket_Strip_Straight_1x12_Pitch2.54mm
- R4, R5: moved to F.Cu
- U1: footprint TO_SOT_Packages_THT:TO-220_Neutral123_Vertical -> TO_SOT_Packages_THT:TO-220-3_Vertical
- moved SW1 41.2 mm to (200.5, 78.5), turned to 270 degrees
- moved C9 25.4 mm to (166.4, 70.6), turned to 90 degrees
- moved Cin1 22.1 mm to (112.8, 95.5), turned to 90 degrees
- moved CON2 17.6 mm to (199.4, 95.0), turned to 0 degrees
- moved L1 16.4 mm to (128.5, 93.0), turned to 270 degrees
- moved D37 15.6 mm to (196.4, 69.6), turned to 0 degrees
- moved R5 11.9 mm to (203.9, 69.6), turned to 0 degrees
- moved R4 11.1 mm to (203.9, 54.9), turned to 0 degrees
- moved Cout1 10.2 mm to (99.6, 91.4)
- moved C8 9.58 mm to (177.5, 96.5), turned to 180 degrees
- moved P11 9.28 mm to (188.2, 101.1), turned to 270 degrees
- moved P9 8.64 mm to (134.1, 67.1), turned to 90 degrees
- moved P10 8.08 mm to (170.7, 67.1), turned to 90 degrees
- moved P15 8.04 mm to (188.2, 109.7)
- moved C7 6.53 mm to (159.8, 96.5), turned to 0 degrees
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Connections:
- CON2 pad 3: (no net) -> Net-(CON2-Pad3)
- P7 pad 1: (no net) -> /TX
- P7 pad 2: (no net) -> /RX
- P7 pad 3: (no net) -> GND
- P7 pad 4: (no net) -> 5V
Routing:
- net GND: track 74.4 -> 16.8 mm
- net 12V: track 188.1 -> 230.3 mm
- net Net-(R1-Pad1): track 26.5 -> 0.00 mm
- net /TX: track 95.9 -> 72.8 mm, vias 1 -> 0
- net /A0: track 47.0 -> 58.5 mm
- net /RX: track 97.8 -> 87.6 mm, vias 1 -> 0
- net 5V: track 360.2 -> 350.6 mm, vias 2 -> 0
- net 24V: track 188.7 -> 198.3 mm, vias 2 -> 0
- net /RST: track 68.9 -> 76.8 mm
- net /D2: track 36.8 -> 30.6 mm
- net /A7: track 32.7 -> 38.9 mm
- net /D7: track 47.8 -> 53.2 mm
- net /A5: track 34.7 -> 38.9 mm
- net /MOSI: track 80.7 -> 84.4 mm, vias 0 -> 1
- net /A1: track 45.5 -> 49.1 mm
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- removed copper zone on B.Cu, net GND
Other:
- board text added: "0"
- board text added: "1"
- board text added: "12V"
- board text added: "2"
- board text added: "24V"
- board text added: "3"
- board text added: "4"
- board text added: "5"
- board text added: "6"
- board text added: "7"
- board text added: "A0"
- board text added: "A1"
- board text added: "A2"
- board text added: "A3"
- board text added: "A4"
- board text added: "A5"
- board text added: "A6"
- board text added: "A7"
- board text added: "B0"
- board text added: "B1"
- board text added: "B2"
- board text added: "B3"
- board text added: "B4"
- board text added: "B5"
- board text added: "B6"
- board text added: "B7"
- board text added: "C0"
- board text added: "C1"
- board text added: "C2"
- board text added: "C3"
- board text added: "C4"
- board text added: "C5"
- board text added: "C6"
- board text added: "C7"
- board text added: "D0"
- board text added: "D1"
- board text added: "D2"
- board text added: "D3"
- board text added: "D4"
- board text added: "D5"
- board text added: "D6"
- board text added: "D7"
- board text added: "PORT A"
- board text added: "Schottky"
