File: Resources/OpenPLCVersion2/KiCAD_Files/Main_Board/OpenPLC_V2.sch (KiCad schematic (older format))
At the start: 42 parts, among them CON1 BARREL_JACK, CON2 AVR-ISP-10, IC1 ATMEGA16-P, J1 Conn_01x04, J2 Conn_01x04, J3 Conn_01x04, J4 Conn_01x04, P10 PortC_B, P11 PortD_B, P12 PortA_M, P13 PortB_M, P14 PortC_M, P15 PortD_M, P3 PortA, P4 PortB, P5 PortC, P6 PortD, P7 Max232, P8 PortB_B, P9 PortA_B, SW1 SW_PUSH, U1 7805, Y1 16Mhz

Commit message: versioning and finalised V 1.3
Parts:
- removed 1N5822: D_Schottky, Diodes_THT:D_DO-201_P12.70mm_Horizontal, symbol D_Schottky
- removed CON1: BARREL_JACK, Connectors:BARREL_JACK, symbol Barrel_Jack
- removed P3: PortA, Terminal_Blocks:TerminalBlock_Pheonix_MKDS1.5-12pol, symbol Conn_01x12
- removed R1, R2: R, Resistors_THT:R_Axial_DIN0207_L6.3mm_D2.5mm_P10.16mm_Horizontal, symbol R
- removed Reg1: LM2596, TO_SOT_Packages_THT:TO-220-5_Vertical, symbol LM2596
- added D3: MBR340, Diodes_THT:D_DO-201AD_P15.24mm_Horizontal, symbol Diode:MBR340
- added D4: D_Schottky, Diodes_THT:D_DO-201AD_P12.70mm_Horizontal, symbol OpenPLC_V2-rescue:D_Schottky-Device
- added J5: Screw_Terminal_01x04, TerminalBlocks_Phoenix:TerminalBlock_Phoenix_MKDS1.5-4pol, symbol Connector:Screw_Terminal_01x04
- added J6: Screw_Terminal_01x08, TerminalBlocks_Phoenix:TerminalBlock_Phoenix_MKDS1.5-8pol, symbol Connector:Screw_Terminal_01x08
- added Regulator1: 24 to 12, TO_SOT_Packages_THT:TO-220-5_Horizontal, symbol Regulator_Switching:LM2576HVT-12
- added powerIn1: 24V, TerminalBlocks_Phoenix:TerminalBlock_Phoenix_MKDS1.5-2pol, symbol OpenPLC_V2-rescue:Screw_Terminal_01x02-Connector
- C2, C3: symbol CP -> OpenPLC_V2-rescue:CP
- C7, C8: symbol CP1 -> OpenPLC_V2-rescue:CP1
- C9: symbol C_Small -> OpenPLC_V2-rescue:C_Small
- CON2: footprint Connect:IDC_Header_Straight_10pins -> IDC:IDC-Header_2x05_Pitch2.54mm_Straight; symbol AVR-ISP-10 -> OpenPLC_V2-rescue:AVR-ISP-10
- Cin1: value CP -> 100uf; symbol CP -> Device:CP
- Cout1: value CP -> 1000uf; footprint Capacitors_THT:CP_Radial_D8.0mm_P3.50mm -> Capacitors_THT:CP_Radial_D10.0mm_P5.00mm; symbol CP -> Device:CP
- D1: footprint Diodes_ThroughHole:Diode_DO-41_SOD81_Horizontal_RM10 -> Diodes_THT:D_DO-41_SOD81_P10.16mm_Horizontal; symbol D -> OpenPLC_V2-rescue:D
- D2, D36, D37: symbol LED-RESCUE-OpenPLC_Kicad_Single_Strip_Unordered -> OpenPLC_Kicad_Single_Strip_Unordered-rescue:LED-RESCUE-OpenPLC_Kicad_Single_Strip_Unordered
- IC1: symbol ATMEGA16-P-RESCUE-OpenPLC_Modular -> OpenPLC_Modular-rescue:ATMEGA16-P-RESCUE-OpenPLC_Modular
- J1, J2, J3, J4: symbol Conn_01x04 -> OpenPLC_V2-rescue:Conn_01x04
- L1: footprint Choke_Axial_ThroughHole:Choke_Horizontal_RM10mm -> Inductors_SMD:L_Fastron_PISR_Handsoldering; symbol INDUCTOR -> OpenPLC_V2-rescue:INDUCTOR
- P10, P11, P8: footprint Socket_Strips:Socket_Strip_Straight_1x08 -> Socket_Strips:Socket_Strip_Straight_1x08_Pitch2.54mm; symbol Conn_01x08 -> OpenPLC_V2-rescue:Conn_01x08
- P12: footprint Pin_Headers:Pin_Header_Straight_1x12 -> Pin_Headers:Pin_Header_Straight_1x12_Pitch2.54mm; symbol Conn_01x12 -> OpenPLC_V2-rescue:Conn_01x12
- P13, P14, P15: footprint Pin_Headers:Pin_Header_Straight_1x08 -> Pin_Headers:Pin_Header_Straight_1x08_Pitch2.54mm; symbol Conn_01x08 -> OpenPLC_V2-rescue:Conn_01x08
- P4, P5, P6: footprint Terminal_Blocks:TerminalBlock_Pheonix_MKDS1.5-8pol -> TerminalBlocks_Phoenix:TerminalBlock_Phoenix_MKDS1.5-8pol; symbol Conn_01x08 -> OpenPLC_V2-rescue:Conn_01x08
- P7: footprint Socket_Strips:Socket_Strip_Angled_1x04 -> Socket_Strips:Socket_Strip_Angled_1x04_Pitch2.54mm; symbol Conn_01x04 -> OpenPLC_V2-rescue:Conn_01x04
- P9: footprint Socket_Strips:Socket_Strip_Straight_1x12 -> Socket_Strips:Socket_Strip_Straight_1x12_Pitch2.54mm; symbol Conn_01x12 -> OpenPLC_V2-rescue:Conn_01x12
- R3: symbol R -> OpenPLC_V2-rescue:R
- R4, R5: symbol R_Small -> OpenPLC_V2-rescue:R_Small
- SW1: symbol SW_PUSH -> OpenPLC_V2-rescue:SW_PUSH
- U1: footprint TO_SOT_Packages_THT:TO-220_Neutral123_Vertical -> TO_SOT_Packages_THT:TO-220-3_Vertical; symbol 7805-RESCUE-OpenPLC_Kicad_Single_Strip_Unordered -> OpenPLC_Kicad_Single_Strip_Unordered-rescue:7805-RESCUE-OpenPLC_Kicad_Single_Strip_Unordered
- Y1: symbol Crystal -> OpenPLC_V2-rescue:Crystal
Connections:
- wire segments 107 -> 206
Other:
- note added: "Power Regulator - 24 to 12V\n"
- note added: "Power Stage - 12 to 5 V\n"
- note removed: "Power Regulator"
- note removed: "Power Stage"
- moved on the sheet: C2, C3, Cin1, D1, D2, D36, D37, J1, J2, J3, J4, L1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
