File: Resources/OpenPLCv2/openPlc_Rpi.kicad_pcb (KiCad board)
At the start: 2 copper layers, 155 x 108 mm, 108 parts, among them J1 Raspberry_Pi_2_3, J10 Conn_01x04, J11 Conn_01x04, J12 Conn_01x04, J13 Conn_01x04, J2 Screw_Terminal_01x05, J3 Screw_Terminal_01x04, J4 Screw_Terminal_01x02, J5 Screw_Terminal_01x12, J6 Screw_Terminal_01x05, J7 Screw_Terminal_01x12, J8 Screw_Terminal_01x02, J9 Screw_Terminal_01x02, K1 G5LE-1, K2 G5LE-1, K3 G5LE-1, K4 G5LE-1, K5 G5LE-1, K6 G5LE-1, K7 G5LE-1, K8 G5LE-1, Q1 BSS123, U1 power_LM2576, U2 LTV-847, U3 LTV-847, U4 power_L7812_smd, U5 MAX481E, U6 ADS1018IDGS, U7 AMS1117-3.3, U8 ULN2803A

Commit message: unknown changes!
Parts:
- removed J2, J6: Screw_Terminal_01x05, TerminalBlocks_Phoenix:TerminalBlock_Phoenix_MKDS1.5-5pol
- removed R46, R47, R48, R49: 50R, Resistor_SMD:R_0805_2012Metric_Pad1.15x1.40mm_HandSolder
- added J14: Screw_Terminal_01x10, TerminalBlock_Phoenix:TerminalBlock_Phoenix_MKDS-1,5-10_1x10_P5.00mm_Horizontal, F.Cu at (131.2, 53.1)
Connections:
- U6 pad 1: Net-(R46-Pad2) -> SCK
- U6 pad 10: Net-(R47-Pad2) -> MOSI
- U6 pad 2: Net-(R49-Pad2) -> CS0
- U6 pad 9: Net-(R48-Pad2) -> MISO
Routing:
- net GND: track 106.4 -> 113.7 mm
Other:
- board text added: "+24V"
- board text added: "A"
- board text added: "B"
- board text added: "GND"
- board text added: "Relay 1"
- board text added: "Relay 2"
- board text added: "Relay 3"
- board text added: "Relay 4"
- board text added: "Relay 5"
- board text added: "Relay 6"
- board text added: "Relay 7"
- board text added: "Relay 8"
- board text added: "SCL"
- board text added: "SDA"
